File: Meter_End_Unit/Meter_End_Unit.kicad_sch (KiCad schematic)
At the start: 12 parts, among them J17 Screw_Terminal_01x01, J18 Screw_Terminal_01x01, J19 Screw_Terminal_01x01, J20 Screw_Terminal_01x01, J6 Jack-DC, U3 BD00FC0WEFJ

Commit message: Update in footprint
Parts:
- 100uf2, 10uf3, 10uf4, C1: footprint Capacitor_SMD:C_0603_1608Metric -> Capacitor_SMD:C_0805_2012Metric
Changed lines of the file:
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@@
 			)
 		)
-		(property "Footprint" "Capacitor_SMD:C_0603_1608Metric"
+		(property "Footprint" "Capacitor_SMD:C_0805_2012Metric"
 			(at 134.3152 53.34 0)
 			(effects
@@
 			)
 		)
-		(property "Footprint" "Capacitor_SMD:C_0603_1608Metric"
+		(property "Footprint" "Capacitor_SMD:C_0805_2012Metric"
 			(at 98.7552 158.75 0)
 			(effects
@@
 			)
 		)
-		(property "Footprint" "Capacitor_SMD:C_0603_1608Metric"
+		(property "Footprint" "Capacitor_SMD:C_0805_2012Metric"
 			(at 135.5852 158.75 0)
 			(effects
@@
 			)
 		)
-		(property "Footprint" "Capacitor_SMD:C_0603_1608Metric"
+		(property "Footprint" "Capacitor_SMD:C_0805_2012Metric"
 			(at 154.6352 53.34 0)
 			(effects
