File: Meter_End_Unit/Meter_End_Unit V2.kicad_pcb (KiCad board)
At the start: 4 copper layers, 150.7 x 71.9 mm, 83 parts, among them J1 Screw_Terminal_01x02, J15 Screw_Terminal_01x01, J16 Screw_Terminal_01x01, J17 Screw_Terminal_01x01, J18 Screw_Terminal_01x01, J19 Screw_Terminal_01x01, J2 Screw_Terminal_01x02, J20 Screw_Terminal_01x01, J21 Screw_Terminal_01x01, J22 Screw_Terminal_01x01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

Commit message: PCB design for meter
Parts:
- moved R20 6.21 mm to (192.9, 102.8), turned to 0 degrees
- moved C26 6.01 mm to (185.5, 102.6), turned to 0 degrees
- moved C27 5.17 mm to (189.3, 105.4), turned to 180 degrees
- moved R10 4.77 mm to (185.2, 105.7), turned to 0 degrees
- moved R11 4.71 mm to (189.2, 102.7), turned to 0 degrees
- moved C38 0.09 mm to (175.2, 131.3)
Routing:
- net GND: track 139.3 -> 108.6 mm, vias 26 -> 29
- net Net-(U5-IAP): track 43.3 -> 30.8 mm, vias 2 -> 0
- net +3.3V: track 34.7 -> 29.6 mm, vias 8 -> 5
- net Net-(U5-IAN): track 32.1 -> 29.1 mm
- net Net-(J1-Pin_1): track 8.32 -> 11.3 mm
- net Net-(J1-Pin_2): track 7.87 -> 5.44 mm
- net Net-(D2-A): track 2.33 -> 0.00 mm
- net Net-(D3-A): track 2.30 -> 0.00 mm
- net +12V: track 21.7 -> 22.7 mm, vias 1 -> 2
- net /ESP32/MISO: track 67.4 -> 68.3 mm
- net Net-(U5-IBN): track 28.2 -> 28.9 mm, vias 2 -> 3
- net Net-(U5-REFIN/OUT): track 9.00 -> 9.52 mm
- net +5V: vias 5 -> 4
Other:
- outline, holes or cut-outs redrawn
