File: Prod_Energy_Theft/Prod_Pole_End_Unit/Prod_Pole_End_Unit.kicad_pcb (KiCad board)
At the start: 2 copper layers, 150 parts, among them IC1 MP1584EN-LF-Z, J14 U.FL-R-SMT_01_, J17 Screw_Terminal_01x02, J18 Screw_Terminal_01x02, J19 Screw_Terminal_01x02, J20 Screw_Terminal_01x02, J21 Screw_Terminal_01x02, J22 Screw_Terminal_01x02, J23 U.FL-R-SMT_01_, J28 JAE_SIM_Card_SF72S006, J6 Jack-DC, J7 SS-52400-002, Q10 BC817, Q2 2N3904, Q9 BC817, U1 TPS7A2033PDBVR, U10 TPS54331DG4, U13 USBLC6-2SC6, U14 E32-433T20S, U15 CP2102N-Axx-xQFN20, U16 ESP32-C6-MINI-1, U17 TXS0108EPW, U18 SIM7600G, U19 ADE7816ACPZ, U2 AP2112K-3.3, U20 USBLC6-2SC6, U21 USBLC6-2SC6, Y3 Crystal

Commit message: PCB Design
Parts:
- moved C76 147.5 mm to (50.7, 90.5), turned to 90 degrees
- moved J22 145.6 mm to (53.6, 100.0)
- moved C92 144.1 mm to (152.3, 71.7)
- moved R86 143.1 mm to (53.2, 90.5), turned to 90 degrees
- moved R95 142.1 mm to (152.2, 74.2)
- moved R94 140.6 mm to (152.1, 76.7), turned to 0 degrees
- moved R93 138.3 mm to (152.1, 79.5)
- moved C77 137.8 mm to (56.1, 90.6), turned to 90 degrees
- moved R90 135.4 mm to (152.2, 87.7), turned to 0 degrees
- moved C2 134.9 mm to (152.3, 90.0), turned to 180 degrees
- moved R87 133.3 mm to (58.6, 90.6), turned to 90 degrees
- moved U17 129.9 mm to (149.5, 58.0)
- moved R83 128.8 mm to (61.1, 90.6), turned to 90 degrees
- moved R84 123.1 mm to (152.3, 99.8)
- moved C69 121.3 mm to (35.8, 90.5), turned to 90 degrees
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Connections:
- 100uf2 pad 2: +5V -> GND
- 1uf1 pad 2: +5V -> GND
- 4.7uf1 pad 2: +5V -> GND
- C1 pad 2: +5V -> GND
- C10 pad 2: +5V -> GND
- C12 pad 2: +5V -> GND
- C13 pad 2: +5V -> GND
- C2 pad 1: +5V -> GND
- C21 pad 2: +5V -> GND
- C24 pad 2: +5V -> GND
- C5 pad 2: +5V -> GND
- C50 pad 2: +5V -> GND
- C51 pad 2: +5V -> GND
- C55 pad 2: +5V -> GND
- C56 pad 1: +5V -> GND
- C57 pad 1: +5V -> GND
- C58 pad 2: +5V -> GND
- C59 pad 2: +5V -> GND
- C60 pad 2: +5V -> GND
- C61 pad 2: +5V -> GND
- C63 pad 1: +5V -> GND
- C64 pad 1: +5V -> GND
- C65 pad 1: +5V -> GND
- C66 pad 1: +5V -> GND
- C67 pad 1: +5V -> GND
- C68 pad 1: +5V -> GND
- C69 pad 1: +5V -> GND
- C7 pad 1: +5V -> GND
- C70 pad 1: +5V -> GND
- C71 pad 1: +5V -> GND
- C72 pad 1: +5V -> GND
- C73 pad 2: +5V -> GND
- C76 pad 1: +5V -> GND
- C77 pad 1: +5V -> GND
- C78 pad 2: +5V -> GND
- C79 pad 2: +5V -> GND
- C80 pad 2: +5V -> GND
- C81 pad 1: +5V -> GND
- C82 pad 2: +5V -> GND
- C83 pad 2: +5V -> GND
- C84 pad 2: +5V -> GND
- C85 pad 2: +5V -> GND
- C86 pad 2: +5V -> GND
- C87 pad 2: +5V -> GND
- C88 pad 2: +5V -> GND
- C89 pad 2: +5V -> GND
- C9 pad 2: +5V -> GND
- C90 pad 2: +5V -> GND
- C91 pad 1: +5V -> GND
- C92 pad 2: +5V -> GND
- C93 pad 1: +5V -> GND
- D2 pad 2: +5V -> GND
- D5 pad 2: +5V -> GND
- IC1 pad 5: +5V -> GND
- IC1 pad 9: +5V -> GND
- J14 pad 1: +5V -> GND
- J14 pad 2: +5V -> GND
- J17 pad 2: +5V -> GND
- J18 pad 2: +5V -> GND
- J19 pad 2: +5V -> GND
- J20 pad 2: +5V -> GND
- J21 pad 2: +5V -> GND
- J22 pad 2: +5V -> GND
- J23 pad 1: +5V -> GND
- J23 pad 2: +5V -> GND
- J28 pad C5: +5V -> GND
- J28 pad SH: +5V -> GND
- J6 pad 2: +5V -> GND
- J7 pad A1: +5V -> GND
- J7 pad A12: +5V -> GND
- J7 pad B1: +5V -> GND
- J7 pad B12: +5V -> GND
- J7 pad G1: +5V -> GND
- J7 pad G2: +5V -> GND
- J7 pad G3: +5V -> GND
- J7 pad G4: +5V -> GND
- J7 pad S1: +5V -> GND
- J7 pad S2: +5V -> GND
- J7 pad S3: +5V -> GND
- J7 pad S4: +5V -> GND
- Q2 pad 1: +5V -> GND
- R13 pad 2: +5V -> GND
- R14 pad 2: +5V -> GND
- R15 pad 2: +5V -> GND
- R16 pad 2: +5V -> GND
- R2 pad 2: +5V -> GND
- R29 pad 1: +5V -> GND
- R56 pad 2: +5V -> GND
- R57 pad 2: +5V -> GND
- R58 pad 2: +5V -> GND
- R6 pad 2: +5V -> GND
- R65 pad 2: +5V -> GND
- R66 pad 2: +5V -> GND
- R67 pad 2: +5V -> GND
- R68 pad 2: +5V -> GND
- R69 pad 2: +5V -> GND
- R71 pad 1: +5V -> GND
- R73 pad 1: +5V -> GND
- R75 pad 1: +5V -> GND
- R77 pad 1: +5V -> GND
- R79 pad 1: +5V -> GND
- R8 pad 2: +5V -> GND
- R83 pad 2: +5V -> GND
- R86 pad 1: +5V -> GND
- R92 pad 1: +3.3V -> +3.3V_ADE
- S5 pad 1: +5V -> GND
- S5 pad 2: +5V -> GND
- S6 pad 1: +5V -> GND
- S6 pad 2: +5V -> GND
- U1 pad 2: +5V -> GND
- U10 pad 7: +5V -> GND
- U13 pad 2: +5V -> GND
- U14 pad 11: +5V -> GND
- U14 pad 13: +5V -> GND
- U14 pad 14: +5V -> GND
- U14 pad 15: +5V -> GND
- U14 pad 16: +5V -> GND
- U14 pad 19: +5V -> GND
- U14 pad 2: +5V -> GND
- U14 pad 26: +5V -> GND
- U14 pad 8: +5V -> GND
- U15 pad 12: +5V -> GND
- U15 pad 21: +5V -> GND
- U15 pad 3: +5V -> GND
- U16 pad 1: +5V -> GND
- U16 pad 11: +5V -> GND
- U16 pad 14: +5V -> GND
- U16 pad 2: +5V -> GND
- U16 pad 36: +5V -> GND
- U16 pad 37: +5V -> GND
- U16 pad 38: +5V -> GND
- U16 pad 39: +5V -> GND
- U16 pad 40: +5V -> GND
- U16 pad 41: +5V -> GND
- U16 pad 42: +5V -> GND
- U16 pad 43: +5V -> GND
- U16 pad 44: +5V -> GND
- U16 pad 45: +5V -> GND
- U16 pad 46: +5V -> GND
- U16 pad 47: +5V -> GND
- U16 pad 48: +5V -> GND
- U16 pad 49: +5V -> GND
- U16 pad 50: +5V -> GND
- U16 pad 51: +5V -> GND
- U16 pad 52: +5V -> GND
- U16 pad 53: +5V -> GND
- U17 pad 11: +5V -> GND
- U18 pad 1: +5V -> GND
- U18 pad 10: +5V -> GND
- U18 pad 110: +5V -> GND
- U18 pad 118: +5V -> GND
- U18 pad 120: +5V -> GND
- U18 pad 121: +5V -> GND
- U18 pad 122: +5V -> GND
- U18 pad 123: +5V -> GND
- U18 pad 124: +5V -> GND
- U18 pad 125: +5V -> GND
- U18 pad 126: +5V -> GND
- U18 pad 127: +5V -> GND
- U18 pad 128: +5V -> GND
- U18 pad 129: +5V -> GND
- U18 pad 130: +5V -> GND
- U18 pad 131: +5V -> GND
- U18 pad 132: +5V -> GND
- U18 pad 133: +5V -> GND
- U18 pad 134: +5V -> GND
- U18 pad 135: +5V -> GND
- U18 pad 14: +5V -> GND
- U18 pad 2: +5V -> GND
- U18 pad 37: +5V -> GND
- U18 pad 40: +5V -> GND
- U18 pad 41: +5V -> GND
- U18 pad 43: +5V -> GND
- U18 pad 5: +5V -> GND
- U18 pad 57: +5V -> GND
- U18 pad 58: +5V -> GND
- U18 pad 60: +5V -> GND
- U18 pad 61: +5V -> GND
- U18 pad 64: +5V -> GND
- U18 pad 65: +5V -> GND
- U18 pad 77: +5V -> GND
- U18 pad 78: +5V -> GND
- U18 pad 80: +5V -> GND
- U18 pad 81: +5V -> GND
- U18 pad 93: +5V -> GND
- U18 pad 98: +5V -> GND
- U19 pad 1: +5V -> GND
- U19 pad 10: +5V -> GND
- U19 pad 11: +5V -> GND
- U19 pad 20: +5V -> GND
- U19 pad 21: +5V -> GND
- U19 pad 25: +5V -> GND
- U19 pad 3: +5V -> GND
- U19 pad 30: +5V -> GND
- U19 pad 31: +5V -> GND
- U19 pad 40: +5V -> GND
- U19 pad 41: +5V -> GND
- U19 pad 6: +5V -> GND
- U2 pad 2: +5V -> GND
- U20 pad 2: +5V -> GND
- U20 pad 5: +5V -> GND
- U21 pad 2: +5V -> GND
- U21 pad 5: +5V -> GND
Routing:
- net GND: track 0.00 -> 592.0 mm, vias 0 -> 61
- net +3.3V: track 0.00 -> 176.1 mm, vias 0 -> 13
- net +V_SIM: track 0.00 -> 154.1 mm, vias 0 -> 4
- net +5V: track 0.00 -> 132.1 mm, vias 0 -> 4
- net /ESP33/DTR: track 0.00 -> 123.4 mm, vias 0 -> 4
- net ESP_PWRKEY: track 0.00 -> 107.7 mm, vias 0 -> 2
- net /ESP33/RTS: track 0.00 -> 107.7 mm, vias 0 -> 4
- net /ESP33/ADE7816/IN: track 0.00 -> 106.3 mm
- net /ESP33/MOSI/SDA: track 0.00 -> 90.0 mm, vias 0 -> 3
- net /ESP33/MISO: track 0.00 -> 82.3 mm, vias 0 -> 4
- net /ESP33/CS: track 0.00 -> 82.0 mm, vias 0 -> 2
- net /ESP33/SCLK/SCL: track 0.00 -> 78.0 mm, vias 0 -> 2
- net /ESP33/RES: track 0.00 -> 75.5 mm, vias 0 -> 2
- net /ESP33/IRQ: track 0.00 -> 74.8 mm, vias 0 -> 2
- net /ESP33/ADE7816/IFP: track 0.00 -> 68.4 mm
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- added copper zone on In2.Cu, net +12V
- added copper zone on In2.Cu, net +3.3V
- added copper zone on In2.Cu, net +3.3V_ADE
- added copper zone on In2.Cu, net +5V
- added copper zone on In2.Cu, net +V_SIM
- added copper zone on In2.Cu, net /VBUS
- added copper zone on In1.Cu, net GND
Other:
- board outline added: 155.4 x 77.8 mm
- copper layers 2 -> 4
